File: Sega Pro.kicad_pcb (KiCad board)
At the start: 2 copper layers, 83.5 x 61.2 mm, 15 parts, among them J1 Game Cartridge Connector, J2 System Edge Connector, SW1 SW_SPDT, U1 27C256, U2 27C256, U3 HY62256ALJ-10, U4 HY62256ALJ-10, U5 LZ95F45

Commit message: Add files via upload
Routing:
- net /SRAM.EN: track 74.7 -> 120.9 mm, vias 4 -> 2
- net /D3: track 145.3 -> 187.4 mm
- net /A5: track 175.9 -> 136.7 mm, vias 7 -> 4
- net /D5: track 135.9 -> 168.0 mm, vias 5 -> 4
- net /D4: track 172.6 -> 149.8 mm, vias 1 -> 6
- net /A11: track 178.4 -> 156.0 mm, vias 7 -> 6
- net //CE_0: track 141.9 -> 123.5 mm, vias 6 -> 2
- net /EEPROM.OE: track 53.0 -> 70.2 mm, vias 4 -> 3
- net /Pwr.Good: track 82.8 -> 66.6 mm, vias 2 -> 4
- net /A9: track 191.2 -> 176.2 mm, vias 7 -> 9
- net /A14: track 180.6 -> 165.7 mm, vias 3 -> 5
- net /D1: track 120.9 -> 135.1 mm, vias 3 -> 5
- net /GND: track 286.4 -> 300.5 mm, vias 13 -> 7
- net /A21: track 62.4 -> 76.5 mm
- net /D10: track 92.2 -> 78.6 mm
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Other:
- board text added: "Codes On Codes Off Trainer"
